Commit message: "Maze_Solver_Complete_Commit"

File: bumperbot_description/urdf/bumperbot.urdf.xacro (robot description, xacro)
@@ -1,4 +1,7 @@
 <?xml version="1.0"?>
 <robot name="bumperbot" xmlns:xacro="http://ros.org/wiki/xacro">
+  <xacro:include filename="common_properties.xacro" />
+  <xacro:include filename="camera.xacro" />
+  <xacro:include filename="lidar.xacro" />
   <!-- Start GZ or Ignition depending on ROS 2 Version -->
   <xacro:arg name="is_ignition" default="true"/>
@@ -23,4 +26,5 @@
         <mesh filename="package://bumperbot_description/meshes/base_link.STL" />
       </geometry>
+      <material name="red" />
     </visual>
     <collision>
@@ -49,4 +53,5 @@
         <mesh filename="package://bumperbot_description/meshes/wheel_right_link.STL" />
       </geometry>
+      <material name="red" />
     </visual>
     <collision>
@@ -77,4 +82,5 @@
         <mesh filename="package://bumperbot_description/meshes/wheel_left_link.STL" />
       </geometry>
+      <material name="red" />
     </visual>
     <collision>
@@ -104,4 +110,5 @@
         <mesh filename="package://bumperbot_description/meshes/caster_front_link.STL" />
       </geometry>
+      <material name="red" />
     </visual>
     <collision>
@@ -131,4 +138,5 @@
         <mesh filename="package://bumperbot_description/meshes/caster_rear_link.STL" />
       </geometry>
+      <material name="red" />
     </visual>
     <collision>

File: bumperbot_description/urdf/bumperbot_gazebo.xacro (robot description, xacro)
@@ -3,4 +3,5 @@
   <!-- Wheels -->
   <gazebo reference="wheel_left_link">
+    <material>Gazebo/Red</material>
     <mu1>1000000000000000.0</mu1>
     <mu2>1000000000000000.0</mu2>
@@ -12,4 +13,5 @@
   </gazebo>
   <gazebo reference="wheel_right_link">
+    <material>Gazebo/Red</material>
     <mu1>1000000000000000.0</mu1>
     <mu2>1000000000000000.0</mu2>
@@ -22,4 +24,5 @@
   <!-- Caster Wheels -->
   <gazebo reference="caster_rear_link">
+    <material>Gazebo/Red</material>
     <mu1>0.1</mu1>
     <mu2>0.1</mu2>
@@ -30,4 +33,5 @@
   </gazebo>
   <gazebo reference="caster_front_link">
+    <material>Gazebo/Red</material>
     <mu1>0.1</mu1>
     <mu2>0.1</mu2>
@@ -44,6 +48,5 @@
         <parameters>$(find bumperbot_controller)/config/bumperbot_controllers.yaml</parameters>
       </plugin>
-      <plugin filename="ignition-gazebo-imu-system" name="ignition::gazebo::systems::Imu">
-      </plugin>
+      <plugin filename="ignition-gazebo-imu-system" name="ignition::gazebo::systems::Imu"></plugin>
     </xacro:if>
     <!-- ROS 2 Iron or above -->
@@ -58,4 +61,5 @@
   <!-- IMU -->
   <gazebo reference="imu_link">
+    <material>Gazebo/Red</material>
     <sensor name="imu" type="imu">
         <always_on>true</always_on>
